File: cansat-pcb/buzzer.kicad_sch (KiCad schematic)
At the start: 8 parts, among them Q1 2N3904, Q2 AO3400A

Commit message: pcb V2
Connections:
- net GND: now also Q2.2 (S); no longer Q2.3 (D)
- net at R1.1: now also Q2.3 (D); no longer Q2.2 (S)
Other:
- moved on the sheet: Q2, R4, R5
Changed lines of the file:
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@@
   (junction (at 152.4 99.06) (diameter 0) (color 0 0 0 0)
   )
+  (junction (at 134.62 88.9) (diameter 0) (color 0 0 0 0)
+  )
   (junction (at 167.64 63.5) (diameter 0) (color 0 0 0 0)
   )
-  (junction (at 134.62 109.22) (diameter 0) (color 0 0 0 0)
-  )
   (wire (pts (xy 152.4 93.98) (xy 168.91 93.98))
     (stroke (width 0) (type default))
@@
     (stroke (width 0) (type default))
   )
-  (wire (pts (xy 118.11 109.22) (xy 121.92 109.22))
+  (wire (pts (xy 134.62 76.2) (xy 134.62 78.74))
     (stroke (width 0) (type default))
   )
@@
     (stroke (width 0) (type default))
   )
-  (wire (pts (xy 134.62 119.38) (xy 134.62 121.92))
-    (stroke (width 0) (type default))
-  )
   (wire (pts (xy 152.4 109.22) (xy 152.4 99.06))
     (stroke (width 0) (type default))
@@
     (stroke (width 0) (type default))
   )
-  (wire (pts (xy 134.62 121.92) (xy 133.35 121.92))
-    (stroke (width 0) (type default))
-  )
   (wire (pts (xy 149.86 99.06) (xy 152.4 99.06))
     (stroke (width 0) (type default))
   )
-  (wire (pts (xy 134.62 109.22) (xy 134.62 111.76))
-    (stroke (width 0) (type default))
-  )
-  (wire (pts (xy 134.62 106.68) (xy 134.62 109.22))
-    (stroke (width 0) (type default))
-  )
-  (wire (pts (xy 129.54 109.22) (xy 134.62 109.22))
-    (stroke (width 0) (type default))
-  )
   (wire (pts (xy 189.23 82.55) (xy 189.23 109.22))
     (stroke (width 0) (type default))
@@
     (stroke (width 0) (type default))
   )
+  (wire (pts (xy 135.89 76.2) (xy 134.62 76.2))
+    (stroke (width 0) (type default))
+  )
   (wire (pts (xy 157.48 63.5) (xy 161.29 63.5))
     (stroke (width 0) (type default))
@@
     (stroke (width 0) (type default))
   )
+  (wire (pts (xy 134.62 86.36) (xy 134.62 88.9))
+    (stroke (width 0) (type default))
+  )
   (wire (pts (xy 189.23 72.39) (xy 189.23 63.5))
     (stroke (width 0) (type default))
@@
     (stroke (width 0) (type default))
   )
+  (wire (pts (xy 134.62 88.9) (xy 134.62 91.44))
+    (stroke (width 0) (type default))
+  )
   (wire (pts (xy 167.64 77.47) (xy 173.99 77.47))
     (stroke (width 0) (type default))
   )
+  (wire (pts (xy 134.62 88.9) (xy 139.7 88.9))
+    (stroke (width 0) (type default))
+  )
   (wire (pts (xy 161.29 63.5) (xy 161.29 91.44))
     (stroke (width 0) (type default))
@@
     (stroke (width 0) (type default))
   )
-  (hierarchical_label "BUZZER" (shape input) (at 133.35 121.92 180) (fields_autoplaced)
-    (effects (font (size 1.27 1.27)) (justify right))
-  )
-  (symbol (lib_id "power:GND") (at 118.11 109.22 270) (unit 1)
-    (in_bom yes) (on_board yes) (dnp no) (fields_autoplaced)
-    (property "Reference" "#PWR020" (at 111.76 109.22 0)
-      (effects (font (size 1.27 1.27)) hide)
-    )
-    (property "Value" "GND" (at 114.3 109.22 90)
+  (hierarchical_label "BUZZER" (shape input) (at 135.89 76.2 0) (fields_autoplaced)
+    (effects (font (size 1.27 1.27)) (justify left))
+  )
+  (symbol (lib_id "power:GND") (at 147.32 88.9 90) (unit 1)
+    (in_bom yes) (on_board yes) (dnp no) (fields_autoplaced)
+    (property "Reference" "#PWR020" (at 153.67 88.9 0)
+      (effects (font (size 1.27 1.27)) hide)
+    )
+    (property "Value" "GND" (at 151.13 88.9 90)
       (effects (font (size 1.27 1.27)) (justify right))
     )
-    (property "Footprint" "" (at 118.11 109.22 0)
-      (effects (font (size 1.27 1.27)) hide)
-    )
-    (property "Datasheet" "" (at 118.11 109.22 0)
+    (property "Footprint" "" (at 147.32 88.9 0)
+      (effects (font (size 1.27 1.27)) hide)
+    )
+    (property "Datasheet" "" (at 147.32 88.9 0)
       (effects (font (size 1.27 1.27)) hide)
     )
@@
     )
   )
-  (symbol (lib_id "Device:R") (at 125.73 109.22 90) (unit 1)
-    (in_bom yes) (on_board yes) (dnp no) (fields_autoplaced)
-    (property "Reference" "R4" (at 125.73 102.87 90)
-      (effects (font (size 1.27 1.27)))
-    )
-    (property "Value" "100K" (at 125.73 105.41 90)
-      (effects (font (size 1.27 1.27)))
-    )
-    (property "Footprint" "Resistor_SMD:R_0805_2012Metric_Pad1.20x1.40mm_HandSolder" (at 125.73 110.998 90)
-      (effects (font (size 1.27 1.27)) hide)
-    )
-    (property "Datasheet" "~" (at 125.73 109.22 0)
+  (symbol (lib_id "Device:R") (at 143.51 88.9 270) (unit 1)
+    (in_bom yes) (on_board yes) (dnp no) (fields_autoplaced)
+    (property "Reference" "R4" (at 143.51 95.25 90)
+      (effects (font (size 1.27 1.27)))
+    )
+    (property "Value" "100K" (at 143.51 92.71 90)
+      (effects (font (size 1.27 1.27)))
+    )
+    (property "Footprint" "Resistor_SMD:R_0805_2012Metric_Pad1.20x1.40mm_HandSolder" (at 143.51 87.122 90)
+      (effects (font (size 1.27 1.27)) hide)
+    )
+    (property "Datasheet" "~" (at 143.51 88.9 0)
       (effects (font (size 1.27 1.27)) hide)
     )
@@
     )
   )
-  (symbol (lib_id "Device:R") (at 134.62 115.57 0) (unit 1)
-    (in_bom yes) (on_board yes) (dnp no) (fields_autoplaced)
-    (property "Reference" "R5" (at 137.16 114.3 0)
-      (effects (font (size 1.27 1.27)) (justify left))
-    )
-    (property "Value" "1K" (at 137.16 116.84 0)
-      (effects (font (size 1.27 1.27)) (justify left))
-    )
-    (property "Footprint" "Resistor_SMD:R_0805_2012Metric_Pad1.20x1.40mm_HandSolder" (at 132.842 115.57 90)
-      (effects (font (size 1.27 1.27)) hide)
-    )
-    (property "Datasheet" "~" (at 134.62 115.57 0)
+  (symbol (lib_id "Device:R") (at 134.62 82.55 180) (unit 1)
+    (in_bom yes) (on_board yes) (dnp no) (fields_autoplaced)
+    (property "Reference" "R5" (at 132.08 83.82 0)
+      (effects (font (size 1.27 1.27)) (justify left))
+    )
+    (property "Value" "1K" (at 132.08 81.28 0)
+      (effects (font (size 1.27 1.27)) (justify left))
+    )
+    (property "Footprint" "Resistor_SMD:R_0805_2012Metric_Pad1.20x1.40mm_HandSolder" (at 136.398 82.55 90)
+      (effects (font (size 1.27 1.27)) hide)
+    )
+    (property "Datasheet" "~" (at 134.62 82.55 0)
       (effects (font (size 1.27 1.27)) hide)
     )
@@
     )
   )
-  (symbol (lib_id "Transistor_FET:AO3400A") (at 134.62 101.6 90) (unit 1)
-    (in_bom yes) (on_board yes) (dnp no) (fields_autoplaced)
-    (property "Reference" "Q2" (at 134.62 92.71 90)
-      (effects (font (size 1.27 1.27)))
-    )
-    (property "Value" "AO3400A" (at 134.62 95.25 90)
-      (effects (font (size 1.27 1.27)))
-    )
-    (property "Footprint" "Package_TO_SOT_SMD:SOT-23" (at 136.525 96.52 0)
+  (symbol (lib_id "Transistor_FET:AO3400A") (at 134.62 96.52 270) (unit 1)
+    (in_bom yes) (on_board yes) (dnp no) (fields_autoplaced)
+    (property "Reference" "Q2" (at 134.62 105.41 90)
+      (effects (font (size 1.27 1.27)))
+    )
+    (property "Value" "AO3400A" (at 134.62 102.87 90)
+      (effects (font (size 1.27 1.27)))
+    )
+    (property "Footprint" "Package_TO_SOT_SMD:SOT-23" (at 132.715 101.6 0)
       (effects (font (size 1.27 1.27) italic) (justify left) hide)
     )
-    (property "Datasheet" "http://www.aosmd.com/pdfs/datasheet/AO3400A.pdf" (at 134.62 101.6 0)
+    (property "Datasheet" "http://www.aosmd.com/pdfs/datasheet/AO3400A.pdf" (at 134.62 96.52 0)
       (effects (font (size 1.27 1.27)) (justify left) hide)
     )
