File: cansat-pcb/cansat pcb.kicad_sch (KiCad schematic)
At the start: 19 parts, among them J1 Conn_01x03_Pin, J2 Conn_01x03_Pin, J3 Conn_01x03_Pin, Q1 2N3904, Q2 AO3400A, SW1 SW_DPDT_x2, U3 MPU6050

Commit message: created MARKDOWN.md
Parts:
- removed J1, J2, J3: Conn_01x03_Pin, Connector_PinHeader_1.00mm:PinHeader_1x03_P1.00mm_Vertical, symbol Connector:Conn_01x03_Pin
- removed M1: ~, CanSat:PowerBoost, symbol CanSat:adafruit_PowerBoost_1000c
- removed Q1: 2N3904, Package_TO_SOT_THT:TO-92_Inline, symbol Transistor_BJT:2N3904
- removed Q2: AO3400A, Package_TO_SOT_SMD:SOT-23, symbol Transistor_FET:AO3400A
- removed R1, R5: 1K, Resistor_SMD:R_0805_2012Metric_Pad1.20x1.40mm_HandSolder, symbol Device:R
- removed R2: 22K, Resistor_SMD:R_0805_2012Metric_Pad1.20x1.40mm_HandSolder, symbol Device:R
- removed R3, R4: 100K, Resistor_SMD:R_0805_2012Metric_Pad1.20x1.40mm_HandSolder, symbol Device:R
- removed S1: ~, CanSat:BMP280, symbol CanSat:BMP280
- removed U1: ~, CanSat:RFM69HCW, symbol CanSat:RFM69HCW
- removed U2: ~, CanSat:KPEG132, symbol CanSat:KPEG132
- removed U3: MPU6050, CanSat:MPU6050, symbol CanSat:MPU6050
- removed U4, U5: ~, Package_TO_SOT_THT:TO-92L_Inline, symbol CanSat:TMP36
Connections:
- net TMP1: now reaches MCU1.31 (GP26)
- net BUZZER: no longer names the net of MCU1.32 (GP27)
- net I2C1 SCL: no longer names the net of MCU1.25 (GP19)
- net I2C1 SDA: no longer names the net of MCU1.24 (GP18)
- net SERVO_1 renamed SERVO/SERVO 1
- net SERVO_2 renamed SERVO/SERVO 2
- net SERVO_3 renamed SERVO/SERVO 3
- net TMP36_1: no longer names the net of MCU1.27 (GP21)
- net TMP36_2 renamed buzzer
Other:
- added sheet BATTERY (BATTERY.kicad_sch)
- added sheet BME688 (BMP280.kicad_sch)
- added sheet BUZZER (buzzer.kicad_sch)
- added sheet CO2 & VOCs (untitled.kicad_sch)
- added sheet GYRO (GYRO.kicad_sch)
- added sheet RADIO (RADIO.kicad_sch)
- added sheet SERVO (servo.kicad_sch)
- added sheet TEMPERATURE (TEMPERATURE.kicad_sch)
- moved on the sheet: SW1A

Commit message: made some changes to pcb (fuck you Berenger)
Parts:
- added J1: Conn_01x02_Pin, Connector_PinHeader_2.54mm:PinHeader_1x02_P2.54mm_Vertical, symbol Connector:Conn_01x02_Pin
- SW1: footprint Connector_PinHeader_1.00mm:PinHeader_1x03_P1.00mm_Vertical -> Connector_PinHeader_2.54mm:PinHeader_1x03_P2.54mm_Vertical
Connections:
- net +5V: now also J1.1 (Pin_1)
- net GND: now also J1.2 (Pin_2)
Other:
- sheet BME688 renamed BMP280
Changed lines of the file:
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@@
+    )
+  )
+  (symbol (lib_id "power:+5V") (at 162.56 93.98 270) (unit 1)
+    (in_bom yes) (on_board yes) (dnp no) (fields_autoplaced)
+    (property "Reference" "#PWR026" (at 158.75 93.98 0)
+      (effects (font (size 1.27 1.27)) hide)
+    )
+    (property "Value" "+5V" (at 166.37 93.98 90)
+      (effects (font (size 1.27 1.27)) (justify left))
+    )
+    (property "Footprint" "" (at 162.56 93.98 0)
+      (effects (font (size 1.27 1.27)) hide)
+    )
+    (property "Datasheet" "" (at 162.56 93.98 0)
+      (effects (font (size 1.27 1.27)) hide)
+    )
+    (pin "1")
+    (instances
+      (project "cansat pcb"
+        (path "/5b536bad-dff4-4fc1-b4ee-d4495f6592c9"
+          (reference "#PWR026") (unit 1)
+        )
+      )
     )
   )
@@
       (effects (font (size 1.27 1.27)))
     )
-    (property "Footprint" "Connector_PinHeader_1.00mm:PinHeader_1x03_P1.00mm_Vertical" (at 190.5 60.96 0)
+    (property "Footprint" "Connector_PinHeader_2.54mm:PinHeader_1x03_P2.54mm_Vertical" (at 190.5 60.96 0)
       (effects (font (size 1.27 1.27)) hide)
     )
@@
     )
   )
+  (symbol (lib_id "power:GND") (at 162.56 96.52 90) (unit 1)
+    (in_bom yes) (on_board yes) (dnp no) (fields_autoplaced)
+    (property "Reference" "#PWR027" (at 168.91 96.52 0)
+      (effects (font (size 1.27 1.27)) hide)
+    )
+    (property "Value" "GND" (at 166.37 96.52 90)
+      (effects (font (size 1.27 1.27)) (justify right))
+    )
+    (property "Footprint" "" (at 162.56 96.52 0)
+      (effects (font (size 1.27 1.27)) hide)
+    )
+    (property "Datasheet" "" (at 162.56 96.52 0)
+      (effects (font (size 1.27 1.27)) hide)
+    )
+    (pin "1")
+    (instances
+      (project "cansat pcb"
+        (path "/5b536bad-dff4-4fc1-b4ee-d4495f6592c9"
+          (reference "#PWR027") (unit 1)
+        )
+      )
+    )
+  )
+  (symbol (lib_id "Connector:Conn_01x02_Pin") (at 157.48 93.98 0) (unit 1)
+    (in_bom yes) (on_board yes) (dnp no) (fields_autoplaced)
+    (property "Reference" "J1" (at 158.115 88.9 0)
+      (effects (font (size 1.27 1.27)))
+    )
+    (property "Value" "Conn_01x02_Pin" (at 158.115 91.44 0)
+      (effects (font (size 1.27 1.27)))
+    )
+    (property "Footprint" "Connector_PinHeader_2.54mm:PinHeader_1x02_P2.54mm_Vertical" (at 157.48 93.98 0)
+      (effects (font (size 1.27 1.27)) hide)
+    )
+    (property "Datasheet" "~" (at 157.48 93.98 0)
+      (effects (font (size 1.27 1.27)) hide)
+    )
+    (pin "1")
+    (pin "2")
+    (instances
+      (project "cansat pcb"
+        (path "/5b536bad-dff4-4fc1-b4ee-d4495f6592c9"
+          (reference "J1") (unit 1)
+        )
+      )
+    )
+  )
   (sheet (at 49.53 63.5) (size 33.02 10.16) (fields_autoplaced)
     (stroke (width 0.1524) (type solid))
@@
     (stroke (width 0.1524) (type solid))
     (fill (color 0 0 0 0.0000))
-    (property "Sheetname" "BME688" (at 49.53 52.6284 0)
-      (effects (font (size 1.27 1.27)) (justify left bottom))
-    )
+    (property "Sheetname" "BMP280" (at 49.53 52.6284 0)
+      (effects (font (size 1.27 1.27)) (justify left bottom))
+    )

Commit message: pcb V2
Connections:
- net CS: now also MCU1.7 (GP5); no longer MCU1.14 (GP5)
- net I2C0 SCL: now also MCU1.2 (GP1); no longer MCU1.19 (GP1)
- net I2C0 SDA: now also MCU1.1 (GP0); no longer MCU1.20 (GP0)
- net MISO: now also MCU1.6 (GP4); no longer MCU1.12 (GP6)
- net MOSI: now also MCU1.10 (GP7); no longer MCU1.11 (GP7)
- net RST: now also MCU1.5 (GP3); no longer MCU1.16 (GP3)
- net SCK: now also MCU1.9 (GP6); no longer MCU1.15 (GP4)
- net SERVO/SERVO 1: now also MCU1.16 (GP12); no longer MCU1.5 (GP12)
- net SERVO/SERVO 2: now also MCU1.15 (GP11); no longer MCU1.6 (GP11)
- net SERVO/SERVO 3: now also MCU1.14 (GP10); no longer MCU1.7 (GP10)
- net VBUS: now reaches MCU1.40 (VBUS)
- new net I2C1 SCL: MCU1.12 (GP9)
- new net I2C1 SDA: MCU1.11 (GP8)
Changed lines of the file:
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@@
     )
   )
-  (global_label "MISO" (shape input) (at 95.25 55.88 180) (fields_autoplaced)
+  (global_label "I2C1 SDA" (shape input) (at 95.25 60.96 180) (fields_autoplaced)
     (effects (font (size 1.27 1.27)) (justify right))
-    (property "Intersheetrefs" "${INTERSHEET_REFS}" (at 87.6686 55.88 0)
+    (property "Intersheetrefs" "${INTERSHEET_REFS}" (at 84.0895 60.96 0)
+      (effects (font (size 1.27 1.27)) (justify right) hide)
+    )
+  )
+  (global_label "I2C1 SCL" (shape input) (at 95.25 63.5 180) (fields_autoplaced)
+    (effects (font (size 1.27 1.27)) (justify right))
+    (property "Intersheetrefs" "${INTERSHEET_REFS}" (at 84.15 63.5 0)
+      (effects (font (size 1.27 1.27)) (justify right) hide)
+    )
+  )
+  (global_label "MISO" (shape input) (at 95.25 50.8 180) (fields_autoplaced)
+    (effects (font (size 1.27 1.27)) (justify right))
+    (property "Intersheetrefs" "${INTERSHEET_REFS}" (at 87.6686 50.8 0)
       (effects (font (size 1.27 1.27)) (justify right) hide)
     )
@@
     )
   )
+  (global_label "VBUS" (shape input) (at 118.11 45.72 0) (fields_autoplaced)
+    (effects (font (size 1.27 1.27)) (justify left))
+    (property "Intersheetrefs" "${INTERSHEET_REFS}" (at 125.3396 45.72 0)
+      (effects (font (size 1.27 1.27)) (justify left) hide)
+    )
+  )
   (global_label "MOSI" (shape input) (at 95.25 58.42 180) (fields_autoplaced)
     (effects (font (size 1.27 1.27)) (justify right))
@@
     )
   )
-  (global_label "SCK" (shape input) (at 95.25 50.8 180) (fields_autoplaced)
+  (global_label "SCK" (shape input) (at 95.25 55.88 180) (fields_autoplaced)
     (effects (font (size 1.27 1.27)) (justify right))
-    (property "Intersheetrefs" "${INTERSHEET_REFS}" (at 88.5153 50.8 0)
+    (property "Intersheetrefs" "${INTERSHEET_REFS}" (at 88.5153 55.88 0)
       (effects (font (size 1.27 1.27)) (justify right) hide)
     )
