File: cansat-pcb/untitled.kicad_sch (KiCad schematic)
At the start: 1 part, among them U5 SGP30

Commit message: made some changes to pcb (fuck you Berenger)
Connections:
- net +3V3: now also U5.1 (VIN); no longer U5.5 (VIN)
- net I2C0 SCL: now also U5.4 (SCL); no longer U5.2 (SCL)
- net I2C0 SDA: now also U5.5 (SDA); no longer U5.1 (SCA)
Other:
- moved on the sheet: U5
Changed lines of the file:
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@@
   (paper "A4")
   (text_box "SGP30\n50mA\n0x58"
-    (at 133.35 88.9 0) (size 40.64 26.67)
+    (at 133.35 88.9 0) (size 44.45 26.67)
     (stroke (width 0) (type default))
     (fill (type none))
     (effects (font (size 1.27 1.27)) (justify left top))
   )
-  (global_label "I2C0 SDA" (shape input) (at 146.05 99.06 180) (fields_autoplaced)
-    (effects (font (size 1.27 1.27)) (justify right))
-    (property "Intersheetrefs" "${INTERSHEET_REFS}" (at 134.2353 99.06 0)
-      (effects (font (size 1.27 1.27)) (justify right) hide)
+  (global_label "I2C0 SCL" (shape input) (at 163.83 101.6 0) (fields_autoplaced)
+    (effects (font (size 1.27 1.27)) (justify left))
+    (property "Intersheetrefs" "${INTERSHEET_REFS}" (at 175.5842 101.6 0)
+      (effects (font (size 1.27 1.27)) (justify left) hide)
     )
   )
-  (global_label "I2C0 SCL" (shape input) (at 146.05 101.6 180) (fields_autoplaced)
-    (effects (font (size 1.27 1.27)) (justify right))
-    (property "Intersheetrefs" "${INTERSHEET_REFS}" (at 134.2958 101.6 0)
-      (effects (font (size 1.27 1.27)) (justify right) hide)
+  (global_label "I2C0 SDA" (shape input) (at 163.83 99.06 0) (fields_autoplaced)
+    (effects (font (size 1.27 1.27)) (justify left))
+    (property "Intersheetrefs" "${INTERSHEET_REFS}" (at 175.6447 99.06 0)
+      (effects (font (size 1.27 1.27)) (justify left) hide)
     )
   )
-  (symbol (lib_id "power:GND") (at 154.94 109.22 0) (unit 1)
+  (symbol (lib_id "power:GND") (at 154.94 106.68 0) (unit 1)
     (in_bom yes) (on_board yes) (dnp no) (fields_autoplaced)
-    (property "Reference" "#PWR025" (at 154.94 115.57 0)
+    (property "Reference" "#PWR025" (at 154.94 113.03 0)
       (effects (font (size 1.27 1.27)) hide)
     )
-    (property "Value" "GND" (at 154.94 114.3 0)
+    (property "Value" "GND" (at 154.94 111.76 0)
       (effects (font (size 1.27 1.27)))
     )
-    (property "Footprint" "" (at 154.94 109.22 0)
+    (property "Footprint" "" (at 154.94 106.68 0)
       (effects (font (size 1.27 1.27)) hide)
     )
-    (property "Datasheet" "" (at 154.94 109.22 0)
+    (property "Datasheet" "" (at 154.94 106.68 0)
       (effects (font (size 1.27 1.27)) hide)
     )
@@
     )
   )
-  (symbol (lib_id "power:+3V3") (at 162.56 101.6 270) (unit 1)
+  (symbol (lib_id "power:+3V3") (at 146.05 99.06 90) (unit 1)
     (in_bom yes) (on_board yes) (dnp no) (fields_autoplaced)
-    (property "Reference" "#PWR024" (at 158.75 101.6 0)
+    (property "Reference" "#PWR024" (at 149.86 99.06 0)
       (effects (font (size 1.27 1.27)) hide)
     )
-    (property "Value" "+3V3" (at 166.37 101.6 90)
+    (property "Value" "+3V3" (at 142.24 99.06 90)
       (effects (font (size 1.27 1.27)) (justify left))
     )
-    (property "Footprint" "" (at 162.56 101.6 0)
+    (property "Footprint" "" (at 146.05 99.06 0)
       (effects (font (size 1.27 1.27)) hide)
     )
-    (property "Datasheet" "" (at 162.56 101.6 0)
+    (property "Datasheet" "" (at 146.05 99.06 0)
       (effects (font (size 1.27 1.27)) hide)
     )

Commit message: pcb V2
Connections:
- net I2C0 SCL renamed I2C1 SCL
- net I2C0 SDA renamed I2C1 SDA
Changed lines of the file:
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@@
     (effects (font (size 1.27 1.27)) (justify left top))
   )
-  (global_label "I2C0 SCL" (shape input) (at 163.83 101.6 0) (fields_autoplaced)
+  (global_label "I2C1 SCL" (shape input) (at 163.83 101.6 0) (fields_autoplaced)
     (effects (font (size 1.27 1.27)) (justify left))
-    (property "Intersheetrefs" "${INTERSHEET_REFS}" (at 175.5842 101.6 0)
+    (property "Intersheetrefs" "${INTERSHEET_REFS}" (at 174.93 101.6 0)
       (effects (font (size 1.27 1.27)) (justify left) hide)
     )
   )
-  (global_label "I2C0 SDA" (shape input) (at 163.83 99.06 0) (fields_autoplaced)
+  (global_label "I2C1 SDA" (shape input) (at 163.83 99.06 0) (fields_autoplaced)
     (effects (font (size 1.27 1.27)) (justify left))
-    (property "Intersheetrefs" "${INTERSHEET_REFS}" (at 175.6447 99.06 0)
+    (property "Intersheetrefs" "${INTERSHEET_REFS}" (at 174.9905 99.06 0)
       (effects (font (size 1.27 1.27)) (justify left) hide)
     )
