File: cansat-pcb/BATTERY.kicad_sch (KiCad schematic)
At the start: 2 parts, among them Q3 DMG2301L

Commit message: V2
Connections:
- no-connect marks 0 -> 1
Changed lines of the file:
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@@
   (junction (at 134.62 115.57) (diameter 0) (color 0 0 0 0)
   )
+  (no_connect (at 105.41 74.93))
   (wire (pts (xy 146.05 87.63) (xy 121.92 87.63))
     (stroke (width 0) (type default))
@@
   )
   (wire (pts (xy 134.62 115.57) (xy 134.62 113.03))
+    (stroke (width 0) (type default))
+  )
+  (wire (pts (xy 121.92 87.63) (xy 121.92 115.57))
     (stroke (width 0) (type default))
   )
@@
     (stroke (width 0) (type default))
   )
-  (wire (pts (xy 121.92 87.63) (xy 121.92 115.57))
-    (stroke (width 0) (type default))
-  )
   (text_box "BATTERY MANAGMENT MODULE"
     (at 99.06 73.66 0) (size 100.33 63.5)
@@
   (global_label "EN_PB" (shape input) (at 153.67 99.06 270) (fields_autoplaced)
     (effects (font (size 1.27 1.27)) (justify right))
-    (property "Intersheetrefs" "${INTERSHEET_REFS}" (at 153.67 108.0323 90)
+    (property "Intersheetrefs" "${INTERSHEET_REFS}" (at 153.67 107.3781 90)
       (effects (font (size 1.27 1.27)) (justify right) hide)
     )
